File: bumble-buzz/schematic_ausf_a/bumble-buzz.kicad_pcb (KiCad board)
At the start: 2 copper layers, 42 parts, among them J1 Conn_01x01_Female, J2 Conn_01x01_Female, Q1 2N2219, Q2 2N2219, Q3 2N2219, Q4 2N2219

Commit message: Intermittent eng thumb redux
Other:
- net class Default removed
